File: MUD-Mesh/MUD-Mesh.kicad_sch (KiCad schematic)
At the start: 9 parts, among them J1 Raspberry_Pi_Zero_2_W, SW1 SW_Push, U1 E22-900M30S, U2 GT-U7

Commit message: feat: power path controller layout started
Parts:
- added C3: 100n, symbol Device:C_Small_US
- added C4: 1u, symbol Device:C_Small_US
- added C5: 100u, symbol Device:C_Small_US
- added D1: PRTR5V0U2X, Package_TO_SOT_SMD:SOT-143, symbol Power_Protection:PRTR5V0U2X
- added D2: ESD9B5.0ST5G, Diode_SMD:D_SOD-923, symbol Diode:ESD9B5.0ST5G
- added F1: PTSLR12106V300, symbol Device:Polyfuse
- added J2: USB_C_Receptacle_USB2.0_14P, symbol Connector:USB_C_Receptacle_USB2.0_14P
- added JP1, JP2, JP3, JP4, JP5, JP6, JP7: SolderJumper_2_Open, symbol Jumper:SolderJumper_2_Open
- added Q1, Q2: NMOS, symbol Simulation_SPICE:NMOS
- added R10: RCharge, symbol Device:R_Small_US
- added R11, R12, R13, R14, R16: 4k, symbol Device:R_Small_US
- added R15: 10m, symbol Device:R_Shunt_US
- added R3: 900k, symbol Device:R_Small_US
- added R4: 4.7k, symbol Device:R_Small_US
- added R5, R6, R8: 200k, symbol Device:R_Small_US
- added R7: 6.2k, symbol Device:R_Small_US
- added R9: 66.5k, symbol Device:R_Small_US
- added U3: TUSB320I, Package_DFN_QFN:Texas_X2QFN-12_1.6x1.6mm_P0.4mm, symbol Interface_USB:TUSB320I
- added U4: LTC4040EUFD, LTC4040EUFD_TRPBF:QFN50P500X400X80-25N, symbol LTC4040EUFD_TRPBF:LTC4040EUFD_TRPBF
Connections:
- net +3V3: now also R5.1, R6.1
- net +5V: now also C3.1, C4.1, C5.1, F1.2, Q1.1 (D), Q2.1 (D), R3.1, R7.1, R8.1, U3.12 (VDD), U4.1 (VSYS), U4.24 (VSYS)
- net GND: now also C3.2, C4.2, C5.2, D1.1 (GND), D2.2 (A2), J2.A1 (GND), J2.A12 (GND), J2.B1 (GND), J2.B12 (GND), J2.S1 (SHIELD), R10.2, R11.2, R12.2, R13.2, R14.2, R16.2, R4.2, R9.2, U3.10 (GND), U3.11 (~{EN}), U3.5 (ADDR), U4.17 (NTC), U4.4 (CHGOFF), U4.5 (BSTOFF)
- net SCL: now also JP2.1 (A), U3.8 (SCL/OUT2); no longer R2.2
- net SDA: now also JP1.1 (A), U3.7 (SDA/OUT1); no longer R1.2
- net USB_CC_INT: now reaches J1.7 (GPCLK0/GPIO04)
- net USB_CC_INT: now also R5.2, U3.6 (~{INT}/OUT3)
- new net: JP2.2 (B), R2.2
- new net: Q1.3 (S), R15.1
- new net: R15.2, U4.6 (VIN)
- new net: R15.3, U4.7 (CLN)
- new net: Q2.3 (S), R15.4
- new net: JP3.1 (A), R14.1
- new net: JP4.1 (A), R13.1
- new net: JP3.2 (B), JP4.2 (B), JP5.2 (B), JP6.2 (B), JP7.2 (B), R10.1, U4.2 (PROG)
- new net: R6.2, U3.9 (ID)
- new net: JP5.1 (A), R12.1
- new net: R7.2, U4.16 (OVSNS)
- new net: JP7.1 (A), R16.1
- new net: JP6.1 (A), R11.1
- new net: D1.2 (I/O1), J2.A5 (CC1), U3.1 (CC1)
- new net: D1.3 (I/O2), J2.B5 (CC2), U3.2 (CC2)
- new net: R4.1, U3.3 (PORT)
- new net: JP1.2 (B), R1.2
- new net: R3.2, U3.4 (VBUS_DET)
- new net: R8.2, R9.1, U4.19 (PFI)
- new net: U4.21 (SW), U4.22 (SW)
- new net IGate: Q1.2 (G), Q2.2 (G), U4.15 (IGATE)
- new net VBUS: D1.4 (VCC), D2.1 (A1), F1.1, J2.A4 (VBUS), J2.A9 (VBUS), J2.B4 (VBUS), J2.B9 (VBUS)
- no-connect marks 1 -> 5
Other:
- moved on the sheet: R1, R2, SW1
